File: 2. Pembuatan Skripsi/2. Alat/1. PCB/Elektronis Pemanas/Elektronis Pemanas.kicad_sch (KiCad schematic)
At the start: 45 parts, among them J1 Conn_02x03_Odd_Even, J2 Conn_01x04, J3 VIN, J4 Sensors, J5 USB_B_Micro, J7 Conn_01x03_Pin, K1 SANYOU_SRD_Form_C, Q1 S8050 JYN, SW3 SW_SPST, U2 AP2112K-3.3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

Commit message: *Merapihkan
*All of the Documents are moved to Laporan
*Numpang folder added
Parts:
- removed D2: LED, LED_SMD:LED_1206_3216Metric_Pad1.42x1.75mm_HandSolder, symbol Device:LED
- removed D6: 1N4001, symbol Device:D_Small
- removed J7: Conn_01x03_Pin, symbol Connector:Conn_01x03_Pin
- removed K1: SANYOU_SRD_Form_C, Relay_THT:Relay_SPDT_SANYOU_SRD_Series_Form_C, symbol Relay:SANYOU_SRD_Form_C
- removed Q1: S8050 JYN, symbol Simulation_SPICE:NPN
- removed R11, R12, R13: 10K, Resistor_SMD:R_0805_2012Metric_Pad1.20x1.40mm_HandSolder, symbol Device:R_Small_US
- removed U3: PC817, Package_DIP:DIP-4_W7.62mm, symbol Isolator:PC817
- added C11: 10uF, Capacitor_SMD:C_0603_1608Metric_Pad1.08x0.95mm_HandSolder, symbol Device:C
- added D1: 1N4148WS, Diode_SMD:D_SOD-323, symbol Diode:1N4148WS
- added D5: LED, LED_SMD:LED_1206_3216Metric_Pad1.42x1.75mm_HandSolder, symbol Device:LED
- added JP1: SolderJumper_2_Open, symbol Jumper:SolderJumper_2_Open
- added K2: EE2-4.5NU, Relay_SMD:Relay_DPDT_Kemet_EE2_NU, symbol Relay:EE2-4.5NU
- added Q1, Q3, Q4: S9013, Package_TO_SOT_SMD:SOT-23, symbol Transistor_BJT:BC850
- added Q2: MMBT2222, Package_TO_SOT_SMD:SOT-23, symbol Transistor_BJT:MMBT3904
- added R2, R5: 10K, Resistor_SMD:R_0805_2012Metric_Pad1.20x1.40mm_HandSolder, symbol Device:R_Small_US
- added R3: 1K, Resistor_SMD:R_0805_2012Metric_Pad1.20x1.40mm_HandSolder, symbol Device:R_Small_US
Connections:
- net GND: now also C11.2, Q2.2 (E), R2.2
- net NRST: now also U5.6 (NRST)
- net RELAYPIN: now also R3.2
- net VCC: now also C11.1, D1.1 (K), K2.1, R5.1
- new net: D5.2 (A), R5.2
- new net: D1.2 (A), JP1.1 (A), K2.12, Q2.3 (C)
- new net: Q2.1 (B), R2.1, R3.1
- new net: D5.1 (K), JP1.2 (B)
- new net COM: K2.9
- new net NC: K2.10
- no-connect marks 1 -> 5
Other:
- note added: "Decouple Cap"
- note added: "EE2-4N3"
- moved on the sheet: C1, C4, C5, C6, C7, J3, J4, R1, U2, U4

Commit message: *New Custom Libs added
- 3631BS Seven segment are added
Parts:
- removed U4: HDSP-A151, Display_7Segment:HDSP-A151, symbol Display_Character:HDSP-A151
- added J6: VIN, Connector:Banana_Jack_2Pin, symbol Connector_Generic:Conn_01x02
- added R11, R12, R17: 1K, Resistor_SMD:R_0603_1608Metric_Pad0.98x0.95mm_HandSolder, symbol Device:R_Small_US
- added R13, R16, R18: 100, Resistor_SMD:R_0603_1608Metric_Pad0.98x0.95mm_HandSolder, symbol Device:R_Small_US
- added R15, R19: 10K, Resistor_SMD:R_0603_1608Metric_Pad0.98x0.95mm_HandSolder, symbol Device:R_Small_US
- added SW1, SW2: SW_SPST, Button_Switch_THT:SW_PUSH_6mm_H13mm, symbol Switch:SW_SPST
- added U3: ~, 3631BS:3631BS 7Segment 3Digit, symbol 3631BS 7Segment 3Digit:3631BS_7_Segment
- C1, C12, C13, C14, C15, C2, C3, C4, C5, C8, C9: footprint Capacitor_SMD:C_0805_2012Metric_Pad1.18x1.45mm_HandSolder -> Capacitor_SMD:C_0603_1608Metric_Pad1.08x0.95mm_HandSolder
- D3: footprint LED_SMD:LED_1206_3216Metric_Pad1.42x1.75mm_HandSolder -> LED_THT:LED_D3.0mm
- D4, D5: footprint LED_SMD:LED_1206_3216Metric_Pad1.42x1.75mm_HandSolder -> LED_SMD:LED_0805_2012Metric_Pad1.15x1.40mm_HandSolder
- J1: footprint (none) -> Connector_IDC:IDC-Header_2x03_P2.54mm_Vertical
- J2: footprint (none) -> Connector_JST:JST_XH_B4B-XH-A_1x04_P2.50mm_Vertical
- J3: footprint (none) -> Connector:Banana_Jack_2Pin
- J4: footprint (none) -> Connector_JST:JST_XH_B3B-XH-A_1x03_P2.50mm_Vertical
- JP1: footprint (none) -> Jumper:SolderJumper-2_P1.3mm_Open_TrianglePad1.0x1.5mm
- R10, R14, R2, R3, R4, R5, R6, R7, R8, R9: footprint Resistor_SMD:R_0805_2012Metric_Pad1.20x1.40mm_HandSolder -> Resistor_SMD:R_0603_1608Metric_Pad0.98x0.95mm_HandSolder
- SW3: footprint Button_Switch_SMD:SW_Push_1P1T_NO_6x6mm_H9.5mm -> Button_Switch_THT:SW_PUSH_6mm_H5mm
- Y3: footprint Crystal:Crystal_HC49-4H_Vertical -> Crystal:Crystal_SMD_HC49-SD
Connections:
- net COM: now also J6.2 (Pin_2)
- net GND: now also J4.3 (Pin_3), R13.2, R15.1, R16.2, R18.2, R19.1
- net NC: now also J6.1 (Pin_1)
- net OSCIN: now also U5.2 (PC14/PB9)
- net OSCOUT: now also U5.3 (PC15)
- net VCC: now also J4.1 (Pin_1), SW1.1 (A), SW2.1 (A)
- net Temp: now reaches J4.2 (Pin_2)
- net Opto: now reaches D1.2 (A), JP1.1 (A), K2.12, Q2.3 (C)
- net at Q1.1 (B): now also R11.1
- net at Q1.2 (E): now also R16.1
- net 1: now reaches Q1.3 (C)
- net 1: now also U3.1
- net at Q3.1 (B): now also R12.1
- net at Q3.2 (E): now also R13.1
- net 2: now reaches Q3.3 (C)
- net 2: now also U3.2
- net at Q4.1 (B): now also R17.1
- net at Q4.2 (E): now also R18.1
- net 3: now reaches Q4.3 (C)
- net 3: now also U3.3
- new net A: U3.A
- new net B: U3.B
- new net C: U3.C
- new net D: U3.D
- new net E: U3.E
- new net EN1: R11.2
- new net EN2: R12.2
- new net EN3: R17.2
- new net F: U3.F
- new net G: U3.G
- new net btn1: R15.2, SW1.2 (B)
- new net btn2: R19.2, SW2.2 (B)
Other:
- note added: "1"
- note added: "10/04/2023"
- note added: "3631BS"
- note added: "7 Segment Display"
- note added: "Heater for Tissue Processor"
- note added: "Pins for DS1820B"
- note added: "Pt Miconos"
- note added: "Push Button"
- note added: "Sensor Pin"
- note added: "To STM"
- note added: "Transistor"
- note added: "Transistor/Optocoupler"
- moved on the sheet: C1, C11, C4, C5, C6, C7, D1, D5, J3, J4, JP1, K2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
