File: 2. Pembuatan Skripsi/2. Alat/1. PCB/Elektronis Pemanas/Elektronis Pemanas.kicad_pcb (KiCad board)
At the start: 2 copper layers, 62.2 x 72.4 mm, 59 parts, among them J1 Conn_02x03_Odd_Even, J2 Conn_01x04, J3 VIN, J4 Sensors, J5 USB_B_Micro, J6 VIN, K2 EE2-4.5NU, Q1 S9013, Q2 MMBT2222, Q3 S9013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

Commit message: First Revision of PCB Design
- Waiting for Approval
Parts:
- Y3: footprint Crystal:Crystal_SMD_HC49-SD_HandSoldering -> Crystal:Crystal_SMD_HC49-SD
Changed lines of the file:
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@@
     )
   )
-  (footprint "Crystal:Crystal_SMD_HC49-SD_HandSoldering" (layer "F.Cu")
+  (footprint "Crystal:Crystal_SMD_HC49-SD" (layer "F.Cu")
     (at 75.438 81.28)
-    (descr "SMD Crystal HC-49-SD http://cdn-reichelt.de/documents/datenblatt/B400/xxx-HC49-SMD.pdf, hand-soldering, 11.4x4.7mm^2 package")
-    (tags "SMD SMT crystal hand-soldering")
+    (descr "SMD Crystal HC-49-SD http://cdn-reichelt.de/documents/datenblatt/B400/xxx-HC49-SMD.pdf, 11.4x4.7mm^2 package")
+    (tags "SMD SMT crystal")
     (property "Sheetfile" "Elektronis Pemanas.kicad_sch")
     (property "Sheetname" "")
@@
         (effects (font (size 1 1) (thickness 0.15)))
     )
-    (fp_line (start -10.075 -2.55) (end -10.075 2.55)
+    (fp_line (start -6.7 -2.55) (end -6.7 2.55)
       (stroke (width 0.12) (type solid)) (layer "F.SilkS"))
-    (fp_line (start -10.075 2.55) (end 5.9 2.55)
+    (fp_line (start -6.7 2.55) (end 5.9 2.55)
       (stroke (width 0.12) (type solid)) (layer "F.SilkS"))
-    (fp_line (start 5.9 -2.55) (end -10.075 -2.55)
+    (fp_line (start 5.9 -2.55) (end -6.7 -2.55)
       (stroke (width 0.12) (type solid)) (layer "F.SilkS"))
-    (fp_line (start -10.2 -2.6) (end -10.2 2.6)
+    (fp_line (start -6.8 -2.6) (end -6.8 2.6)
       (stroke (width 0.05) (type solid)) (layer "F.CrtYd"))
-    (fp_line (start -10.2 2.6) (end 10.2 2.6)
+    (fp_line (start -6.8 2.6) (end 6.8 2.6)
       (stroke (width 0.05) (type solid)) (layer "F.CrtYd"))
-    (fp_line (start 10.2 -2.6) (end -10.2 -2.6)
+    (fp_line (start 6.8 -2.6) (end -6.8 -2.6)
       (stroke (width 0.05) (type solid)) (layer "F.CrtYd"))
-    (fp_line (start 10.2 2.6) (end 10.2 -2.6)
+    (fp_line (start 6.8 2.6) (end 6.8 -2.6)
       (stroke (width 0.05) (type solid)) (layer "F.CrtYd"))
     (fp_line (start -5.7 -2.35) (end -5.7 2.35)
@@
     (fp_arc (start 3.015 -2.115) (mid 5.13 0) (end 3.015 2.115)
       (stroke (width 0.1) (type solid)) (layer "F.Fab"))
-    (pad "1" smd rect (at -5.9375 0) (size 7.875 2) (layers "F.Cu" "F.Paste" "F.Mask")
+    (pad "1" smd rect (at -4.25 0) (size 4.5 2) (layers "F.Cu" "F.Paste" "F.Mask")
       (net 7 "OSCOUT") (pinfunction "1") (pintype "passive"))
-    (pad "2" smd rect (at 5.9375 0) (size 7.875 2) (layers "F.Cu" "F.Paste" "F.Mask")
+    (pad "2" smd rect (at 4.25 0) (size 4.5 2) (layers "F.Cu" "F.Paste" "F.Mask")
       (net 6 "OSCIN") (pinfunction "2") (pintype "passive"))
     (model "${KICAD6_3DMODEL_DIR}/Crystal.3dshapes/Crystal_SMD_HC49-SD.wrl"
