File: 2. Pembuatan Skripsi/2. Alat/1. PCB/ATMEGA328 Version/ATMEGA328 Version/ATMEGA328 Heat Component of Tissue Processor.kicad_sch (KiCad schematic)
At the start: 64 parts, among them J1 Conn_01x02, J2 Sensors, J3 Screw_Terminal_01x02, J5 FTDI, J6 Conn_02x04_Top_Bottom, K1 EE2-4.5NU, Q1 S9013, Q2 S9013, Q3 S9013, Q4 MMBT2222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

Commit message: Huge Update
- New program
- Report updated
Connections:
- net EN2: now also R5.1; no longer R5.2
- net at Q2.1 (B): now also R5.2; no longer R5.1
Other:
- moved on the sheet: R5
Changed lines of the file:
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@@
     )
   )
-  (symbol (lib_id "Device:R_Small_US") (at 173.99 92.964 270) (unit 1)
+  (symbol (lib_id "Device:R_Small_US") (at 173.99 92.964 90) (mirror x) (unit 1)
     (in_bom yes) (on_board yes) (dnp no)
-    (property "Reference" "R5" (at 173.482 91.186 90)
+    (property "Reference" "R5" (at 174.498 91.186 90)
       (effects (font (size 1.27 1.27)))
     )
